Commit message: El filtro funciona adecuadamente. Se le ha agregado ruido a la odometría del apriltag_box, de forma que el filtro no logra dar una salida limpia. El siguiente paso es transformar también la velocidad de la odometría, para que así el filtro pueda ser más robusto.

File: ros_workspace/src/rotors_simulator/rotors_description/urdf/apriltag_box.xacro (robot description, xacro)
@@ -163,12 +163,12 @@
     measurement_delay="0"
     unknown_delay="0.0"
-    noise_normal_position="0 0 0"
-    noise_normal_quaternion="0 0 0"
-    noise_normal_linear_velocity="0 0 0"
-    noise_normal_angular_velocity="0 0 0"
-    noise_uniform_position="0 0 0"
-    noise_uniform_quaternion="0 0 0"
-    noise_uniform_linear_velocity="0 0 0"
-    noise_uniform_angular_velocity="0 0 0"
+    noise_normal_position="0.3 0.3 0.3"
+    noise_normal_quaternion="0.1 0.1 0.1"
+    noise_normal_linear_velocity="0.1 0.1 0.1"
+    noise_normal_angular_velocity="0.05 0.05 0.05"
+    noise_uniform_position="0.3 0.3 0.3"
+    noise_uniform_quaternion="0.1 0.1 0.1"
+    noise_uniform_linear_velocity="0.1 0.1 0.1"
+    noise_uniform_angular_velocity="0.05 0.05 0.05"
     enable_odometry_map="false"
     odometry_map=""

File: ros_workspace/src/rotors_simulator/rotors_description/urdf/camera.xacro (robot description, xacro)
@@ -16,5 +16,7 @@
         <parent link="${namespace}/camera_link"/>
         <child link="${namespace}/camera_link_optical"/>
-        <origin xyz="0.01 0.01 0.01" rpy="0 -1.5708 -1.5708"/>
+        <origin xyz="0.01 0.01 0.01" rpy="-1.5708 0 -1.5708"/>
+        <!-- <origin xyz="0.01 0.01 0.01" rpy="0 0 0"/> -->
+        <!-- <origin xyz="0.01 0.01 0.01" rpy="0 0 0"/> -->
     </joint>
     <link name="${namespace}/camera_link_optical"></link>

Commit message: Latest packages for hardware testing

File: ros_workspace/src/rotors_simulator/rotors_description/urdf/apriltag_box.xacro (robot description, xacro)
@@ -5,5 +5,5 @@
 			<geometry>
 				<!-- <mesh filename="package://blimp_description/meshes/docking/cube_with_apriltags.dae" scale="0.2 0.2 0.2"/> -->
-				<mesh filename="$(find rotors_description)/meshes/cube_with_apriltags.dae" scale="0.2 0.2 0.2"/>
+				<mesh filename="$(find rotors_description)/meshes/cube_with_apriltags.dae" scale="0.1 0.1 0.1"/>
 			</geometry>
 		</visual>
@@ -163,12 +163,12 @@
     measurement_delay="0"
     unknown_delay="0.0"
-    noise_normal_position="1 1 1"
-    noise_normal_quaternion="1 1 1"
-    noise_normal_linear_velocity="1 1 1"
-    noise_normal_angular_velocity="0.5 0.5 0.5"
-    noise_uniform_position="1 1 1"
-    noise_uniform_quaternion="1 1 1"
-    noise_uniform_linear_velocity="1 1 1"
-    noise_uniform_angular_velocity="0.5 0.5 0.5"
+    noise_normal_position="0 0 0"
+    noise_normal_quaternion="0 0 0"
+    noise_normal_linear_velocity="0 0 0"
+    noise_normal_angular_velocity="0 0 0"
+    noise_uniform_position="0 0 0"
+    noise_uniform_quaternion="0 0 0"
+    noise_uniform_linear_velocity="0 0 0"
+    noise_uniform_angular_velocity="0 0 0"
     enable_odometry_map="false"
     odometry_map=""

File: ros_workspace/src/rotors_simulator/rotors_description/urdf/camera.xacro (robot description, xacro)
@@ -11,5 +11,5 @@
         <parent link="${namespace}/base_link"/>
         <child link="${namespace}/camera_link"/>
-        <origin xyz="0.05 0 0.12" rpy="0 0 0"/>
+        <origin xyz="0.088 0 -0.1" rpy="0 0 0"/>
     </joint>
     <joint name="${namespace}/camera_optical_joint" type="fixed">
@@ -28,5 +28,6 @@
             <update_rate>30</update_rate>
             <camera>
-                <horizontal_fov>1.089</horizontal_fov>
+                <!-- <horizontal_fov>1.089</horizontal_fov> -->
+                <horizontal_fov>1.1712319</horizontal_fov>
                 <image>
                     <format>R8G8B8</format>
@@ -35,5 +36,5 @@
                 </image>
                 <clip>
-                    <near>0.09</near>
+                    <near>0.01</near>
                     <far>100</far>
                 </clip>
